File: StripArray.kicad_pcb (KiCad board)
At the start: 2 copper layers, 368 parts, among them U1 WS2811, U10 WS2811, U11 WS2811, U12 WS2811, U13 WS2811, U14 WS2811, U15 WS2811, U16 WS2811, U2 WS2811, U3 WS2811, U4 WS2811, U5 WS2811, U6 WS2811, U7 WS2811, U8 WS2811, U9 WS2811

Commit message: LED Driver array PCB
Parts:
- LedStrip10, LedStrip11, LedStrip12, LedStrip13, LedStrip14, LedStrip15, LedStrip16, LedStrip2, LedStrip3, LedStrip4, LedStrip5, LedStrip6, LedStrip7, LedStrip8, LedStrip9: moved to B.Cu
- moved Qredinv16 293.4 mm to (345.2, 76.0), turned to 90 degrees
- moved Qredout16 291.8 mm to (345.2, 66.2), turned to 90 degrees
- moved Qredinv14 270.5 mm to (303.2, 76.0), turned to 90 degrees
- moved Qredinv15 269.8 mm to (324.2, 76.0), turned to 90 degrees
- moved Qredout14 269.4 mm to (303.2, 66.2), turned to 90 degrees
- moved Qredout15 268.2 mm to (324.2, 66.2), turned to 90 degrees
- moved Qredinv11 230.0 mm to (240.2, 76.0), turned to 90 degrees
- moved Qredout11 230.0 mm to (240.2, 66.2), turned to 90 degrees
- moved Qredinv12 228.4 mm to (261.2, 76.0), turned to 90 degrees
- moved Qredout12 227.8 mm to (261.2, 66.2), turned to 90 degrees
- moved Qredinv13 227.3 mm to (282.2, 76.0), turned to 90 degrees
- moved Qredout13 226.1 mm to (282.2, 66.2), turned to 90 degrees
- moved Qgreenout16 204.7 mm to (340.0, 66.2), turned to 90 degrees
- moved Qgreeninv16 202.7 mm to (340.0, 76.0), turned to 90 degrees
- moved Qblueout16 197.7 mm to (334.8, 66.2), turned to 90 degrees
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
Commit message: Draw borders in silk on PCB
Parts:
- moved Jin5 0.25 mm to (100.2, 64.8)
- moved Jout5 0.25 mm to (117.8, 64.8)
- moved Rvdd10 0.25 mm to (221.5, 93.0)
Other:
- board text added: "DIN"
- board text added: "DOUT"
- board text added: "G"
- board text added: "VDD"

Commit message: Add logotype to silk
Parts:
- added G***: LOGO, StripArray:LedAlertLogotype, B.Cu at (339.2, 75.5)
- added G***: LOGO, StripArray:LedAlertLogotype, B.Cu at (150.2, 75.5)
- added G***: LOGO, StripArray:LedAlertLogotype, B.Cu at (129.2, 75.5)
- added G***: LOGO, StripArray:LedAlertLogotype, B.Cu at (108.2, 75.5)
- added G***: LOGO, StripArray:LedAlertLogotype, B.Cu at (87.2, 75.5)
- added G***: LOGO, StripArray:LedAlertLogotype, B.Cu at (66.2, 75.5)
- added G***: LOGO, StripArray:LedAlertLogotype, B.Cu at (45.2, 75.5)
- added G***: LOGO, StripArray:LedAlertLogotype, B.Cu at (24.2, 75.5)
- added G***: LOGO, StripArray:LedAlertLogotype, B.Cu at (318.2, 75.5)
- added G***: LOGO, StripArray:LedAlertLogotype, B.Cu at (297.2, 75.5)
- added G***: LOGO, StripArray:LedAlertLogotype, B.Cu at (276.2, 75.5)
- added G***: LOGO, StripArray:LedAlertLogotype, B.Cu at (255.2, 75.5)
- added G***: LOGO, StripArray:LedAlertLogotype, B.Cu at (234.2, 75.5)
- added G***: LOGO, StripArray:LedAlertLogotype, B.Cu at (213.2, 75.5)
- added G***: LOGO, StripArray:LedAlertLogotype, B.Cu at (192.2, 75.5)
- added G***: LOGO, StripArray:LedAlertLogotype, B.Cu at (171.2, 75.5)
Other:
- board text added: "Tim Gremalm 2021-01-21 https://github.com/TimGremalm/StripArray"

Commit message: PCB routing
Parts:
- moved Rblueout7 10.5 mm to (145.8, 71.2)
- moved Rredout7 10.5 mm to (156.2, 71.2)
- moved Jin4 5.00 mm to (79.2, 64.8), turned to 180 degrees
Routing:
- net /AddressableLedDriver01/VIn: track 0.00 -> 994.8 mm
- net /AddressableLedDriver01/GndIn: track 0.00 -> 749.5 mm, vias 0 -> 99
- net /AddressableLedDriver12/DIN: track 0.00 -> 78.0 mm
- net /AddressableLedDriver02/DIN: track 0.00 -> 78.0 mm
- net /AddressableLedDriver03/DIN: track 0.00 -> 77.9 mm
- net /AddressableLedDriver04/DIN: track 0.00 -> 77.8 mm
- net /AddressableLedDriver07/DIN: track 0.00 -> 77.5 mm
- net /AddressableLedDriver08/DIN: track 0.00 -> 77.2 mm
- net /AddressableLedDriver14/DIN: track 0.00 -> 77.0 mm
- net /AddressableLedDriver11/DIN: track 0.00 -> 76.8 mm
- net /AddressableLedDriver10/DIN: track 0.00 -> 76.1 mm
- net /AddressableLedDriver15/DIN: track 0.00 -> 75.6 mm
- net /AddressableLedDriver13/DIN: track 0.00 -> 75.4 mm
- net /AddressableLedDriver06/DIN: track 0.00 -> 75.2 mm
- net /AddressableLedDriver09/DIN: track 0.00 -> 75.2 mm
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- added copper zone on B.Cu, net /AddressableLedDriver01/GndIn
Other:
- board outline added: 336 x 40 mm

Commit message: Continued PCB routing
Routing:
- net /AddressableLedDriver01/GndIn: track 749.5 -> 793.1 mm, vias 99 -> 127
- net Net-(C8-Pad1): track 46.4 -> 62.7 mm, vias 0 -> 2
- net Net-(C14-Pad1): track 46.3 -> 62.6 mm, vias 0 -> 2
- net Net-(C13-Pad1): track 45.9 -> 62.0 mm, vias 0 -> 2
- net Net-(C7-Pad1): track 46.0 -> 62.1 mm, vias 0 -> 2
- net Net-(C6-Pad1): track 46.0 -> 62.1 mm, vias 0 -> 2
- net Net-(C15-Pad1): track 46.2 -> 62.3 mm, vias 0 -> 2
- net Net-(C12-Pad1): track 46.1 -> 62.3 mm, vias 0 -> 2
- net Net-(C11-Pad1): track 45.9 -> 62.1 mm, vias 0 -> 2
- net Net-(C9-Pad1): track 46.8 -> 62.9 mm, vias 0 -> 2
- net Net-(C16-Pad1): track 45.8 -> 61.9 mm, vias 0 -> 2
- net Net-(C10-Pad1): track 46.2 -> 62.1 mm, vias 0 -> 2
- net Net-(C4-Pad1): track 47.8 -> 63.7 mm, vias 0 -> 2
- net Net-(C2-Pad1): track 45.8 -> 61.6 mm, vias 0 -> 2
- net Net-(C5-Pad1): track 45.9 -> 61.7 mm, vias 0 -> 2
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
Commit message: Route new headers
Parts:
- removed G*** (x16): LOGO, StripArray:LedAlertLogotype
- removed Rdo1, Rdo10, Rdo11, Rdo12, Rdo13, Rdo14, Rdo15, Rdo16, Rdo2, Rdo3, Rdo4, Rdo5, Rdo6, Rdo7, Rdo8, Rdo9: 33R, Capacitors_SMD:C_0603_HandSoldering
- added Hbottomleft1: MountingHole, Mounting_Holes:MountingHole_3.2mm_M3_Pad, F.Cu at (18.5, 92.5)
- added Hbottomleft10: MountingHole, Mounting_Holes:MountingHole_3.2mm_M3_Pad, F.Cu at (207.5, 92.5)
- added Hbottomleft11: MountingHole, Mounting_Holes:MountingHole_3.2mm_M3_Pad, F.Cu at (228.5, 92.5)
- added Hbottomleft12: MountingHole, Mounting_Holes:MountingHole_3.2mm_M3_Pad, F.Cu at (249.5, 92.5)
- added Hbottomleft13: MountingHole, Mounting_Holes:MountingHole_3.2mm_M3_Pad, F.Cu at (270.5, 92.5)
- added Hbottomleft14: MountingHole, Mounting_Holes:MountingHole_3.2mm_M3_Pad, F.Cu at (291.5, 92.5)
- added Hbottomleft15: MountingHole, Mounting_Holes:MountingHole_3.2mm_M3_Pad, F.Cu at (312.5, 92.5)
- added Hbottomleft16: MountingHole, Mounting_Holes:MountingHole_3.2mm_M3_Pad, F.Cu at (333.5, 92.5)
- added Hbottomleft2: MountingHole, Mounting_Holes:MountingHole_3.2mm_M3_Pad, F.Cu at (39.5, 92.5)
- added Hbottomleft3: MountingHole, Mounting_Holes:MountingHole_3.2mm_M3_Pad, F.Cu at (60.5, 92.5)
- added Hbottomleft4: MountingHole, Mounting_Holes:MountingHole_3.2mm_M3_Pad, F.Cu at (81.5, 92.5)
- added Hbottomleft5: MountingHole, Mounting_Holes:MountingHole_3.2mm_M3_Pad, F.Cu at (102.5, 92.5)
- added Hbottomleft6: MountingHole, Mounting_Holes:MountingHole_3.2mm_M3_Pad, F.Cu at (123.5, 92.5)
- added Hbottomleft7: MountingHole, Mounting_Holes:MountingHole_3.2mm_M3_Pad, F.Cu at (144.5, 92.5)
- added Hbottomleft8: MountingHole, Mounting_Holes:MountingHole_3.2mm_M3_Pad, F.Cu at (165.5, 92.5)
- added Hbottomleft9: MountingHole, Mounting_Holes:MountingHole_3.2mm_M3_Pad, F.Cu at (186.5, 92.5)
- added Jrgb1: Conn_01x04_Female, Pin_Headers:Pin_Header_Straight_1x04_Pitch2.54mm, F.Cu at (30.0, 62.8)
- added Jrgb10: Conn_01x04_Female, Pin_Headers:Pin_Header_Straight_1x04_Pitch2.54mm, F.Cu at (219.0, 62.8)
- added Jrgb11: Conn_01x04_Female, Pin_Headers:Pin_Header_Straight_1x04_Pitch2.54mm, F.Cu at (240.0, 62.8)
- added Jrgb12: Conn_01x04_Female, Pin_Headers:Pin_Header_Straight_1x04_Pitch2.54mm, F.Cu at (261.0, 62.8)
- added Jrgb13: Conn_01x04_Female, Pin_Headers:Pin_Header_Straight_1x04_Pitch2.54mm, F.Cu at (282.0, 62.8)
- added Jrgb14: Conn_01x04_Female, Pin_Headers:Pin_Header_Straight_1x04_Pitch2.54mm, F.Cu at (303.0, 62.8)
- added Jrgb15: Conn_01x04_Female, Pin_Headers:Pin_Header_Straight_1x04_Pitch2.54mm, F.Cu at (324.0, 62.8)
- added Jrgb16: Conn_01x04_Female, Pin_Headers:Pin_Header_Straight_1x04_Pitch2.54mm, F.Cu at (345.0, 62.8)
- added Jrgb2: Conn_01x04_Female, Pin_Headers:Pin_Header_Straight_1x04_Pitch2.54mm, F.Cu at (51.0, 62.8)
- added Jrgb3: Conn_01x04_Female, Pin_Headers:Pin_Header_Straight_1x04_Pitch2.54mm, F.Cu at (72.0, 62.8)
- added Jrgb4: Conn_01x04_Female, Pin_Headers:Pin_Header_Straight_1x04_Pitch2.54mm, F.Cu at (93.0, 62.8)
- added Jrgb5: Conn_01x04_Female, Pin_Headers:Pin_Header_Straight_1x04_Pitch2.54mm, F.Cu at (114.0, 62.8)
- added Jrgb6: Conn_01x04_Female, Pin_Headers:Pin_Header_Straight_1x04_Pitch2.54mm, F.Cu at (135.0, 62.8)
- added Jrgb7: Conn_01x04_Female, Pin_Headers:Pin_Header_Straight_1x04_Pitch2.54mm, F.Cu at (156.0, 62.8)
- added Jrgb8: Conn_01x04_Female, Pin_Headers:Pin_Header_Straight_1x04_Pitch2.54mm, F.Cu at (177.0, 62.8)
- added Jrgb9: Conn_01x04_Female, Pin_Headers:Pin_Header_Straight_1x04_Pitch2.54mm, F.Cu at (198.0, 62.8)
- added Rset1: 0R, Capacitors_SMD:C_0603_HandSoldering, F.Cu at (31.2, 95.2)
- added Rset10: 0R, Capacitors_SMD:C_0603_HandSoldering, F.Cu at (220.2, 95.5)
- added Rset11: 0R, Capacitors_SMD:C_0603_HandSoldering, F.Cu at (241.2, 95.8)
- added Rset12: 0R, Capacitors_SMD:C_0603_HandSoldering, F.Cu at (262.2, 95.8)
- added Rset13: 0R, Capacitors_SMD:C_0603_HandSoldering, F.Cu at (283.2, 95.8)
- added Rset14: 0R, Capacitors_SMD:C_0603_HandSoldering, F.Cu at (304.2, 95.8)
- added Rset15: 0R, Capacitors_SMD:C_0603_HandSoldering, F.Cu at (325.3, 95.8)
- added Rset16: 0R, Capacitors_SMD:C_0603_HandSoldering, F.Cu at (346.0, 95.8)
- added Rset2: 0R, Capacitors_SMD:C_0603_HandSoldering, F.Cu at (52.2, 95.5)
- added Rset3: 0R, Capacitors_SMD:C_0603_HandSoldering, F.Cu at (73.2, 95.5)
- added Rset4: 0R, Capacitors_SMD:C_0603_HandSoldering, F.Cu at (94.2, 95.5)
- added Rset5: 0R, Capacitors_SMD:C_0603_HandSoldering, F.Cu at (115.0, 95.5)
- added Rset6: 0R, Capacitors_SMD:C_0603_HandSoldering, F.Cu at (136.2, 95.8)
- added Rset7: 0R, Capacitors_SMD:C_0603_HandSoldering, F.Cu at (157.2, 95.8)
- added Rset8: 0R, Capacitors_SMD:C_0603_HandSoldering, F.Cu at (178.2, 95.8)
- added Rset9: 0R, Capacitors_SMD:C_0603_HandSoldering, F.Cu at (199.3, 95.8)
- moved Rdin1 2.78 mm to (20.0, 87.5), turned to 180 degrees
- moved Rdin4 2.66 mm to (82.5, 87.2), turned to 180 degrees
- moved Rdin14 2.61 mm to (292.2, 87.0), turned to 180 degrees
- moved Rdin6 2.57 mm to (124.5, 87.0), turned to 180 degrees
- moved Rdin5 2.37 mm to (103.5, 87.2), turned to 180 degrees
- moved Rdin2 2.37 mm to (40.5, 87.2), turned to 180 degrees
- moved Rdin3 2.36 mm to (61.5, 87.2), turned to 180 degrees
- moved Rdin10 2.24 mm to (208.5, 87.2), turned to 180 degrees
- moved Rdin11 2.24 mm to (229.5, 87.2), turned to 180 degrees
- moved Rdin13 2.24 mm to (271.5, 87.2), turned to 180 degrees
- moved Rdin16 2.24 mm to (334.2, 87.2), turned to 180 degrees
- moved Rdin9 2.24 mm to (187.2, 87.2), turned to 180 degrees
- moved Rdin7 2.15 mm to (145.2, 87.5), turned to 180 degrees
- moved Rdin8 2.15 mm to (166.2, 87.5), turned to 180 degrees
- moved Rdin15 2.14 mm to (313.2, 87.2), turned to 180 degrees
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Connections:
- U1 pad 5: Net-(Rdo1-Pad2) -> /AddressableLedDriver02/DIN
- U10 pad 5: Net-(Rdo10-Pad2) -> /AddressableLedDriver11/DIN
- U11 pad 5: Net-(Rdo11-Pad2) -> /AddressableLedDriver12/DIN
- U12 pad 5: Net-(Rdo12-Pad2) -> /AddressableLedDriver13/DIN
- U13 pad 5: Net-(Rdo13-Pad2) -> /AddressableLedDriver14/DIN
- U14 pad 5: Net-(Rdo14-Pad2) -> /AddressableLedDriver15/DIN
- U15 pad 5: Net-(Rdo15-Pad2) -> /AddressableLedDriver16/DIN
- U16 pad 5: Net-(Rdo16-Pad2) -> /AddressableLedDriver16/DOUT
- U2 pad 5: Net-(Rdo2-Pad2) -> /AddressableLedDriver03/DIN
- U3 pad 5: Net-(Rdo3-Pad2) -> /AddressableLedDriver04/DIN
- U4 pad 5: Net-(Rdo4-Pad2) -> /AddressableLedDriver05/DIN
- U5 pad 5: Net-(Rdo5-Pad2) -> /AddressableLedDriver06/DIN
- U6 pad 5: Net-(Rdo6-Pad2) -> /AddressableLedDriver07/DIN
- U7 pad 5: Net-(Rdo7-Pad2) -> /AddressableLedDriver08/DIN
- U8 pad 5: Net-(Rdo8-Pad2) -> /AddressableLedDriver09/DIN
- U9 pad 5: Net-(Rdo9-Pad2) -> /AddressableLedDriver10/DIN
Routing:
- net /AddressableLedDriver01/VIn: track 994.8 -> 1047.0 mm
- net Net-(Rdo1-Pad2): track 8.33 -> 0.00 mm
- net /AddressableLedDriver02/DIN: track 78.0 -> 70.1 mm
- net Net-(Rdo2-Pad2): track 6.93 -> 0.00 mm
- net Net-(Rset9-Pad2): track 0.00 -> 6.31 mm
- net Net-(Rset15-Pad2): track 0.00 -> 6.31 mm
- net Net-(Rset8-Pad2): track 0.00 -> 6.26 mm
- net Net-(Rset7-Pad2): track 0.00 -> 6.26 mm
- net Net-(Rset6-Pad2): track 0.00 -> 6.26 mm
- net Net-(Rset11-Pad2): track 0.00 -> 6.26 mm
- net Net-(Rset16-Pad2): track 0.00 -> 6.26 mm
- net Net-(Rset14-Pad2): track 0.00 -> 6.26 mm
- net Net-(Rset13-Pad2): track 0.00 -> 6.26 mm
- net Net-(Rset12-Pad2): track 0.00 -> 6.26 mm
- net Net-(Rset4-Pad2): track 0.00 -> 6.26 mm
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