File: AddressableLedDriver.sch (KiCad schematic (older format))
At the start: 23 parts, among them U1 WS2811

Commit message: Removed faulty  junction between DIN and GND
Connections:
- net DOUT: no longer C1.2, Jin1.1 (Pin_1), Jout1.1 (Pin_1), Qblueinv1.2 (S), Qblueout1.2 (S), Qgreeninv1.2 (S), Qgreenout1.2 (S), Qredinv1.2 (S), Qredout1.2 (S), U1.4 (GND)
- new net GndIn: C1.2, Jin1.1 (Pin_1), Jout1.1 (Pin_1), Qblueinv1.2 (S), Qblueout1.2 (S), Qgreeninv1.2 (S), Qgreenout1.2 (S), Qredinv1.2 (S), Qredout1.2 (S), U1.4 (GND)
Changed lines of the file:
@@
 	2500 4700 2550 4700
-Wire Wire Line
-	2850 4700 3450 4700
 Wire Wire Line
 	8850 4700 8850 4400
 Wire Wire Line
 	8850 4400 10450 4400
-Connection ~ 3450 4700
-Wire Wire Line
-	3450 4700 8850 4700
 Wire Wire Line
 	10350 4600 10350 2300
@@
 	1    0    0    -1
 $EndComp
+Wire Wire Line
+	2850 4700 8850 4700
 $EndSCHEMATC

Commit message: Comment schematic, titles
Parts:
- added Hbottomleft1, Hbottomright1, Htopleft1, Htopright1: MountingHole, Mounting_Holes:MountingHole_3.2mm_M3_Pad, symbol Mechanical:MountingHole
Other:
- note added: "Match footprint of RGB LED Strip"
- note added: "Use a two stage MOSFET to invert signal."
- note added: "WS2811 hava internal LDO with goal of 5.5V.\nWorldsemi recommends 2.7k in series with VDD to regulate current at 2.40mA.\n(24V-5.5V)/0.00240A = 7708 Ohm\nClosest E12 is 8.2k will put it at 2.25mA."
- note removed: "WS2811 VDD absolute maximum 6.0V"
Changed lines of the file:
@@
 encoding utf-8
 Sheet 2 17
-Title ""
-Date ""
-Rev ""
+Title "Strip Array - LED driver"
+Date "2021-01-23"
+Rev "2021-01-23"
 Comp ""
-Comment1 ""
-Comment2 ""
+Comment1 "WS2811 LED driver with external MOSFET's for RGB."
+Comment2 "https://github.com/TimGremalm/StripArray"
 Comment3 ""
 Comment4 ""
@@
 	1    0    0    -1
 $EndComp
-Text Notes 2600 2450 0    50   ~ 0
-WS2811 VDD absolute maximum 6.0V
+Text Notes 2700 2750 0    50   ~ 0
+WS2811 hava internal LDO with goal of 5.5V.\nWorldsemi recommends 2.7k in series with VDD to regulate current at 2.40mA.\n(24V-5.5V)/0.00240A = 7708 Ohm\nClosest E12 is 8.2k will put it at 2.25mA.
 $Comp
 L Device:R Rgreenout?
@@
 AR Path="/601B7703/601B0CCE" Ref="#FLG013"  Part="1"
 AR Path="/601B7A66/601B0CCE" Ref="#FLG014"  Part="1"
-F 0 "#FLG0103" H 3450 3175 50  0001 C CNN
+F 0 "#FLG014" H 3450 3175 50  0001 C CNN
 F 1 "PWR_FLAG" H 3450 3273 50  0001 C CNN
 F 2 "" H 3450 3100 50  0001 C CNN
@@
 Wire Wire Line
 	2850 4700 8850 4700
+$Comp
+L Mechanical:MountingHole Htopleft1
+U 1 1 600BA38D
+P 3800 6900
+AR Path="/60059F31/600BA38D" Ref="Htopleft1"  Part="1"
+AR Path="/601AD743/600BA38D" Ref="Htopleft2"  Part="1"
+AR Path="/601B6580/600BA38D" Ref="Htopleft11"  Part="1"
+AR Path="/601B4EED/600BA38D" Ref="Htopleft3"  Part="1"
+AR Path="/601B5265/600BA38D" Ref="Htopleft4"  Part="1"
+AR Path="/601B55BF/600BA38D" Ref="Htopleft5"  Part="1"
+AR Path="/601B5793/600BA38D" Ref="Htopleft6"  Part="1"
+AR Path="/601B59D7/600BA38D" Ref="Htopleft7"  Part="1"
+AR Path="/601B5B26/600BA38D" Ref="Htopleft8"  Part="1"
+AR Path="/601B5F54/600BA38D" Ref="Htopleft9"  Part="1"
+AR Path="/601B617C/600BA38D" Ref="Htopleft10"  Part="1"
+AR Path="/601B6B91/600BA38D" Ref="Htopleft12"  Part="1"
+AR Path="/601B714E/600BA38D" Ref="Htopleft13"  Part="1"
+AR Path="/601B73ED/600BA38D" Ref="Htopleft14"  Part="1"
+AR Path="/601B7703/600BA38D" Ref="Htopleft15"  Part="1"
+AR Path="/601B7A66/600BA38D" Ref="Htopleft16"  Part="1"
+F 0 "Htopleft1" H 3900 6946 50  0000 L CNN
+F 1 "MountingHole" H 3900 6855 50  0000 L CNN
+F 2 "Mounting_Holes:MountingHole_3.2mm_M3_Pad" H 3800 6900 50  0001 C CNN
+F 3 "~" H 3800 6900 50  0001 C CNN
+	1    3800 6900
+	1    0    0    -1
+$EndComp
+$Comp
+L Mechanical:MountingHole Htopright1
+U 1 1 600BDC42
+P 4550 6900
+AR Path="/60059F31/600BDC42" Ref="Htopright1"  Part="1"
+AR Path="/601AD743/600BDC42" Ref="Htopright2"  Part="1"
+AR Path="/601B6580/600BDC42" Ref="Htopright11"  Part="1"
+AR Path="/601B4EED/600BDC42" Ref="Htopright3"  Part="1"
+AR Path="/601B5265/600BDC42" Ref="Htopright4"  Part="1"
+AR Path="/601B55BF/600BDC42" Ref="Htopright5"  Part="1"
+AR Path="/601B5793/600BDC42" Ref="Htopright6"  Part="1"
+AR Path="/601B59D7/600BDC42" Ref="Htopright7"  Part="1"
+AR Path="/601B5B26/600BDC42" Ref="Htopright8"  Part="1"
+AR Path="/601B5F54/600BDC42" Ref="Htopright9"  Part="1"
+AR Path="/601B617C/600BDC42" Ref="Htopright10"  Part="1"
+AR Path="/601B6B91/600BDC42" Ref="Htopright12"  Part="1"
+AR Path="/601B714E/600BDC42" Ref="Htopright13"  Part="1"
+AR Path="/601B73ED/600BDC42" Ref="Htopright14"  Part="1"
+AR Path="/601B7703/600BDC42" Ref="Htopright15"  Part="1"
+AR Path="/601B7A66/600BDC42" Ref="Htopright16"  Part="1"
+F 0 "Htopright1" H 4650 6946 50  0000 L CNN
+F 1 "MountingHole" H 4650 6855 50  0000 L CNN
+F 2 "Mounting_Holes:MountingHole_3.2mm_M3_Pad" H 4550 6900 50  0001 C CNN
+F 3 "~" H 4550 6900 50  0001 C CNN
+	1    4550 6900
+	1    0    0    -1
+$EndComp
+$Comp
+L Mechanical:MountingHole Hbottomleft1
+U 1 1 600C04DB
+P 3800 7300
+AR Path="/60059F31/600C04DB" Ref="Hbottomleft1"  Part="1"
+AR Path="/601AD743/600C04DB" Ref="Hbottomleft2"  Part="1"
+AR Path="/601B6580/600C04DB" Ref="Hbottomleft11"  Part="1"
+AR Path="/601B4EED/600C04DB" Ref="Hbottomleft3"  Part="1"
+AR Path="/601B5265/600C04DB" Ref="Hbottomleft4"  Part="1"
+AR Path="/601B55BF/600C04DB" Ref="Hbottomleft5"  Part="1"
+AR Path="/601B5793/600C04DB" Ref="Hbottomleft6"  Part="1"
+AR Path="/601B59D7/600C04DB" Ref="Hbottomleft7"  Part="1"
+AR Path="/601B5B26/600C04DB" Ref="Hbottomleft8"  Part="1"
+AR Path="/601B5F54/600C04DB" Ref="Hbottomleft9"  Part="1"
+AR Path="/601B617C/600C04DB" Ref="Hbottomleft10"  Part="1"
+AR Path="/601B6B91/600C04DB" Ref="Hbottomleft12"  Part="1"
+AR Path="/601B714E/600C04DB" Ref="Hbottomleft13"  Part="1"
+AR Path="/601B73ED/600C04DB" Ref="Hbottomleft14"  Part="1"
+AR Path="/601B7703/600C04DB" Ref="Hbottomleft15"  Part="1"
+AR Path="/601B7A66/600C04DB" Ref="Hbottomleft16"  Part="1"
+F 0 "Hbottomleft1" H 3900 7346 50  0000 L CNN
+F 1 "MountingHole" H 3900 7255 50  0000 L CNN
+F 2 "Mounting_Holes:MountingHole_3.2mm_M3_Pad" H 3800 7300 50  0001 C CNN
+F 3 "~" H 3800 7300 50  0001 C CNN
+	1    3800 7300
+	1    0    0    -1
+$EndComp
+$Comp
+L Mechanical:MountingHole Hbottomright1
+U 1 1 600C2E75
+P 4550 7300
+AR Path="/60059F31/600C2E75" Ref="Hbottomright1"  Part="1"
+AR Path="/601AD743/600C2E75" Ref="Hbottomright2"  Part="1"
+AR Path="/601B6580/600C2E75" Ref="Hbottomright11"  Part="1"
+AR Path="/601B4EED/600C2E75" Ref="Hbottomright3"  Part="1"
+AR Path="/601B5265/600C2E75" Ref="Hbottomright4"  Part="1"
+AR Path="/601B55BF/600C2E75" Ref="Hbottomright5"  Part="1"
+AR Path="/601B5793/600C2E75" Ref="Hbottomright6"  Part="1"
+AR Path="/601B59D7/600C2E75" Ref="Hbottomright7"  Part="1"
+AR Path="/601B5B26/600C2E75" Ref="Hbottomright8"  Part="1"
+AR Path="/601B5F54/600C2E75" Ref="Hbottomright9"  Part="1"
+AR Path="/601B617C/600C2E75" Ref="Hbottomright10"  Part="1"
+AR Path="/601B6B91/600C2E75" Ref="Hbottomright12"  Part="1"
+AR Path="/601B714E/600C2E75" Ref="Hbottomright13"  Part="1"
+AR Path="/601B73ED/600C2E75" Ref="Hbottomright14"  Part="1"
+AR Path="/601B7703/600C2E75" Ref="Hbottomright15"  Part="1"
+AR Path="/601B7A66/600C2E75" Ref="Hbottomright16"  Part="1"
+F 0 "Hbottomright1" H 4650 7346 50  0000 L CNN
+F 1 "MountingHole" H 4650 7255 50  0000 L CNN
+F 2 "Mounting_Holes:MountingHole_3.2mm_M3_Pad" H 4550 7300 50  0001 C CNN
+F 3 "~" H 4550 7300 50  0001 C CNN
+	1    4550 7300
+	1    0    0    -1
+$EndComp
+Text Notes 4850 4200 0    50   ~ 0
+Use a two stage MOSFET to invert signal.
+Text Notes 7200 1600 0    50   ~ 0
+Match footprint of RGB LED Strip
 $EndSCHEMATC

Commit message: Resistor for WS2811 set pin 400/800kHz
Parts:
- removed Rdo1: 33R, Capacitors_SMD:C_0603_HandSoldering, symbol Device:R
- added Rredinv?: 0R, Capacitors_SMD:C_0603_HandSoldering, symbol Device:R
Connections:
- net DOUT: now also U1.5 (DO)
- net at C1.1, Rblueinv1.1, Rblueout1.1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: now also Rredinv?.1
- net at U1.7 (SET): now also Rredinv?.2
- no-connect marks 1 -> 0
Other:
- note added: "Set floating for high speed 800kHz mode.\nSet high for low speed mode 400kHz."
- note added: "WS2811 hava internal LDO with goal of 5.5V.\nWorldsemi recommends 2.7k in series with VDD to regulate current at 2.40mA at 12V.\n(24V-5.5V)/2.40mA = 7.7 kOhm\nClosest E12 is 8.2k will put it at 2.25mA."
- note removed: "WS2811 hava internal LDO with goal of 5.5V.\nWorldsemi recommends 2.7k in series with VDD to regulate current at 2.40mA.\n(24V-5.5V)/0.00240A = 7708 Ohm\nClosest E12 is 8.2k will put it at 2.25mA."
Changed lines of the file:
@@
 $EndComp
-$Comp
-L Device:R Rdo?
-U 1 1 6006C530
-P 2700 4700
-AR Path="/6006C530" Ref="Rdo?"  Part="1"
-AR Path="/60059F31/6006C530" Ref="Rdo1"  Part="1"
-AR Path="/601AD743/6006C530" Ref="Rdo2"  Part="1"
-AR Path="/601B4EED/6006C530" Ref="Rdo3"  Part="1"
-AR Path="/601B5265/6006C530" Ref="Rdo4"  Part="1"
-AR Path="/601B55BF/6006C530" Ref="Rdo5"  Part="1"
-AR Path="/601B5793/6006C530" Ref="Rdo6"  Part="1"
-AR Path="/601B59D7/6006C530" Ref="Rdo7"  Part="1"
-AR Path="/601B5B26/6006C530" Ref="Rdo8"  Part="1"
-AR Path="/601B5F54/6006C530" Ref="Rdo9"  Part="1"
-AR Path="/601B617C/6006C530" Ref="Rdo10"  Part="1"
-AR Path="/601B6580/6006C530" Ref="Rdo11"  Part="1"
-AR Path="/601B6B91/6006C530" Ref="Rdo12"  Part="1"
-AR Path="/601B714E/6006C530" Ref="Rdo13"  Part="1"
-AR Path="/601B73ED/6006C530" Ref="Rdo14"  Part="1"
-AR Path="/601B7703/6006C530" Ref="Rdo15"  Part="1"
-AR Path="/601B7A66/6006C530" Ref="Rdo16"  Part="1"
-F 0 "Rdo1" V 2493 4700 50  0000 C CNN
-F 1 "33R" V 2584 4700 50  0000 C CNN
-F 2 "Capacitors_SMD:C_0603_HandSoldering" V 2630 4700 50  0001 C CNN
-F 3 "~" H 2700 4700 50  0001 C CNN
-	1    2700 4700
-	0    1    1    0
-$EndComp
-NoConn ~ 3050 4500
 $Comp
 L Device:R Rredout?
@@
 	1    0    0    -1
 $EndComp
-$Comp
-L Driver_LED:WS2811 U?
-U 1 1 6006C559
-P 3450 4400
-AR Path="/6006C559" Ref="U?"  Part="1"
-AR Path="/60059F31/6006C559" Ref="U1"  Part="1"
-AR Path="/601AD743/6006C559" Ref="U2"  Part="1"
-AR Path="/601B4EED/6006C559" Ref="U3"  Part="1"
-AR Path="/601B5265/6006C559" Ref="U4"  Part="1"
-AR Path="/601B55BF/6006C559" Ref="U5"  Part="1"
-AR Path="/601B5793/6006C559" Ref="U6"  Part="1"
-AR Path="/601B59D7/6006C559" Ref="U7"  Part="1"
-AR Path="/601B5B26/6006C559" Ref="U8"  Part="1"
-AR Path="/601B5F54/6006C559" Ref="U9"  Part="1"
-AR Path="/601B617C/6006C559" Ref="U10"  Part="1"
-AR Path="/601B6580/6006C559" Ref="U11"  Part="1"
-AR Path="/601B6B91/6006C559" Ref="U12"  Part="1"
-AR Path="/601B714E/6006C559" Ref="U13"  Part="1"
-AR Path="/601B73ED/6006C559" Ref="U14"  Part="1"
-AR Path="/601B7703/6006C559" Ref="U15"  Part="1"
-AR Path="/601B7A66/6006C559" Ref="U16"  Part="1"
-F 0 "U1" H 3450 4850 50  0000 C CNN
-F 1 "WS2811" H 3450 4750 50  0000 C CNN
-F 2 "Housings_SOIC:SOIC-8_3.9x4.9mm_Pitch1.27mm" H 3150 4550 50  0001 C CNN
-F 3 "https://cdn-shop.adafruit.com/datasheets/WS2811.pdf" H 3250 4650 50  0001 C CNN
-	1    3450 4400
-	1    0    0    -1
-$EndComp
 Wire Wire Line
 	4250 3800 4250 3450
@@
 	1    0    0    -1
 $EndComp
-Text Notes 2700 2750 0    50   ~ 0
-WS2811 hava internal LDO with goal of 5.5V.\nWorldsemi recommends 2.7k in series with VDD to regulate current at 2.40mA.\n(24V-5.5V)/0.00240A = 7708 Ohm\nClosest E12 is 8.2k will put it at 2.25mA.
+Text Notes 2350 2150 0    50   ~ 0
+WS2811 hava internal LDO with goal of 5.5V.\nWorldsemi recommends 2.7k in series with VDD to regulate current at 2.40mA at 12V.\n(24V-5.5V)/2.40mA = 7.7 kOhm\nClosest E12 is 8.2k will put it at 2.25mA.
 $Comp
 L Device:R Rgreenout?
@@
 	2500 4400 2500 4700
 Wire Wire Line
-	2500 4700 2550 4700
-Wire Wire Line
 	8850 4700 8850 4400
 Wire Wire Line
@@
 	10450 4400 10500 4400
 Wire Wire Line
-	3450 3100 2350 3100
+	3450 3100 2950 3100
 Connection ~ 3450 3100
 Connection ~ 2350 3100
@@
 AR Path="/601B7703/601B0CCE" Ref="#FLG013"  Part="1"
 AR Path="/601B7A66/601B0CCE" Ref="#FLG014"  Part="1"
-F 0 "#FLG014" H 3450 3175 50  0001 C CNN
+F 0 "#FLG0103" H 3450 3175 50  0001 C CNN
 F 1 "PWR_FLAG" H 3450 3273 50  0001 C CNN
 F 2 "" H 3450 3100 50  0001 C CNN
@@
 	1    0    0    -1
 $EndComp
-Wire Wire Line
-	2850 4700 8850 4700
 $Comp
 L Mechanical:MountingHole Htopleft1
@@
 Text Notes 7200 1600 0    50   ~ 0
 Match footprint of RGB LED Strip
+Wire Wire Line
+	2500 4700 8850 4700
+Connection ~ 2950 3100
+Wire Wire Line
+	2950 3100 2350 3100
+$Comp
+L Driver_LED:WS2811 U?
+U 1 1 6006C559
+P 3450 4400
+AR Path="/6006C559" Ref="U?"  Part="1"
+AR Path="/60059F31/6006C559" Ref="U1"  Part="1"
+AR Path="/601AD743/6006C559" Ref="U2"  Part="1"
+AR Path="/601B4EED/6006C559" Ref="U3"  Part="1"
+AR Path="/601B5265/6006C559" Ref="U4"  Part="1"
+AR Path="/601B55BF/6006C559" Ref="U5"  Part="1"
+AR Path="/601B5793/6006C559" Ref="U6"  Part="1"
+AR Path="/601B59D7/6006C559" Ref="U7"  Part="1"
+AR Path="/601B5B26/6006C559" Ref="U8"  Part="1"
+AR Path="/601B5F54/6006C559" Ref="U9"  Part="1"
+AR Path="/601B617C/6006C559" Ref="U10"  Part="1"
+AR Path="/601B6580/6006C559" Ref="U11"  Part="1"
+AR Path="/601B6B91/6006C559" Ref="U12"  Part="1"
+AR Path="/601B714E/6006C559" Ref="U13"  Part="1"
+AR Path="/601B73ED/6006C559" Ref="U14"  Part="1"
+AR Path="/601B7703/6006C559" Ref="U15"  Part="1"
+AR Path="/601B7A66/6006C559" Ref="U16"  Part="1"
+F 0 "U1" H 3450 4850 50  0000 C CNN
+F 1 "WS2811" H 3450 4750 50  0000 C CNN
+F 2 "Housings_SOIC:SOIC-8_3.9x4.9mm_Pitch1.27mm" H 3150 4550 50  0001 C CNN
+F 3 "https://cdn-shop.adafruit.com/datasheets/WS2811.pdf" H 3250 4650 50  0001 C CNN
+	1    3450 4400
+	1    0    0    -1
+$EndComp
+Wire Wire Line
+	2950 4500 3050 4500
+Wire Wire Line
+	2950 3200 2950 3100
+Wire Wire Line
+	2950 3500 2950 4500
+$Comp
+L Device:R Rredinv?
+U 1 1 600E943A
+P 2950 3350
+AR Path="/600E943A" Ref="Rredinv?"  Part="1"
+AR Path="/60059F31/600E943A" Ref="Rset?"  Part="1"
+AR Path="/601AD743/600E943A" Ref="Rredinv?"  Part="1"
+AR Path="/601B4EED/600E943A" Ref="Rredinv?"  Part="1"
+AR Path="/601B5265/600E943A" Ref="Rredinv?"  Part="1"
+AR Path="/601B55BF/600E943A" Ref="Rredinv?"  Part="1"
+AR Path="/601B5793/600E943A" Ref="Rredinv?"  Part="1"
+AR Path="/601B59D7/600E943A" Ref="Rredinv?"  Part="1"
+AR Path="/601B5B26/600E943A" Ref="Rredinv?"  Part="1"
+AR Path="/601B5F54/600E943A" Ref="Rredinv?"  Part="1"
+AR Path="/601B617C/600E943A" Ref="Rredinv?"  Part="1"
+AR Path="/601B6580/600E943A" Ref="Rredinv?"  Part="1"
+AR Path="/601B6B91/600E943A" Ref="Rredinv?"  Part="1"
+AR Path="/601B714E/600E943A" Ref="Rredinv?"  Part="1"
+AR Path="/601B73ED/600E943A" Ref="Rredinv?"  Part="1"
+AR Path="/601B7703/600E943A" Ref="Rredinv?"  Part="1"
+AR Path="/601B7A66/600E943A" Ref="Rredinv?"  Part="1"
+F 0 "Rset?" H 3020 3396 50  0000 L CNN
+F 1 "0R" H 3020 3305 50  0000 L CNN
+F 2 "Capacitors_SMD:C_0603_HandSoldering" V 2880 3350 50  0001 C CNN
+F 3 "~" H 2950 3350 50  0001 C CNN
+F 4 "DNP" H 2950 3350 50  0001 C CNN "DNP"
+	1    2950 3350
+	1    0    0    -1
+$EndComp
+Text Notes 2950 2950 0    50   ~ 0
+Set floating for high speed 800kHz mode.\nSet high for low speed mode 400kHz.
 $EndSCHEMATC

Commit message: Add extra RGB header
Parts:
- removed Rredinv?: 0R, Capacitors_SMD:C_0603_HandSoldering, symbol Device:R
- added Jrgb1: Conn_01x04_Female, Pin_Headers:Pin_Header_Straight_1x04_Pitch2.54mm, symbol Connector:Conn_01x04_Female
- added Rset1: 0R, Capacitors_SMD:C_0603_HandSoldering, symbol Device:R
Connections:
- net VIn: now also Jrgb1.1 (Pin_1)
- net at C1.1, Rblueinv1.1, Rblueout1.1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: now also Rset1.1
- net at U1.7 (SET): now also Rset1.2
- net at LedStrip1.2 (Pin_2), Qredout1.3 (D): now also Jrgb1.2 (Pin_2)
- net at LedStrip1.3 (Pin_3), Qgreenout1.3 (D): now also Jrgb1.3 (Pin_3)
- net at LedStrip1.4 (Pin_4), Qblueout1.3 (D): now also Jrgb1.4 (Pin_4)

Commit message: Route new headers
Parts:
- removed Hbottomright1, Htopleft1, Htopright1: MountingHole, Mounting_Holes:MountingHole_3.2mm_M3_Pad, symbol Mechanical:MountingHole

Commit message: Add interactive BOM and DNP fields to headers
Parts:
- Hbottomleft1, Jin1, Jout1, Jrgb1, LedStrip1: DNP (none) -> DNP
Changed lines of the file:
@@
 F 2 "StripArray:RGB_Strip" H 7350 1800 50  0001 C CNN
 F 3 "~" H 7350 1800 50  0001 C CNN
+F 4 "DNP" V 7350 1800 50  0001 C CNN "DNP"
 	1    7350 1800
 	0    -1   -1   0
@@
 F 2 "Pin_Headers:Pin_Header_Straight_1x03_Pitch2.54mm" H 10150 4700 50  0001 C CNN
 F 3 "~" H 10150 4700 50  0001 C CNN
+F 4 "DNP" H 10150 4700 50  0001 C CNN "DNP"
 	1    10150 4700
 	-1   0    0    1
@@
 F 2 "Pin_Headers:Pin_Header_Straight_1x03_Pitch2.54mm" H 1700 4700 50  0001 C CNN
 F 3 "~" H 1700 4700 50  0001 C CNN
+F 4 "DNP" H 1700 4700 50  0001 C CNN "DNP"
 	1    1700 4700
 	-1   0    0    1
@@
 AR Path="/601B7703/601B0CCE" Ref="#FLG013"  Part="1"
 AR Path="/601B7A66/601B0CCE" Ref="#FLG014"  Part="1"
-F 0 "#FLG014" H 3450 3175 50  0001 C CNN
+F 0 "#FLG0103" H 3450 3175 50  0001 C CNN
 F 1 "PWR_FLAG" H 3450 3273 50  0001 C CNN
 F 2 "" H 3450 3100 50  0001 C CNN
@@
 F 2 "Mounting_Holes:MountingHole_3.2mm_M3_Pad" H 3800 7300 50  0001 C CNN
 F 3 "~" H 3800 7300 50  0001 C CNN
+F 4 "DNP" H 3800 7300 50  0001 C CNN "DNP"
 	1    3800 7300
 	1    0    0    -1
@@
 F 2 "Pin_Headers:Pin_Header_Straight_1x04_Pitch2.54mm" H 7350 1300 50  0001 C CNN
 F 3 "~" H 7350 1300 50  0001 C CNN
+F 4 "DNP" V 7350 1300 50  0001 C CNN "DNP"
 	1    7350 1300
 	0    -1   -1   0
